File: solenoid-led-strip/solenoid-led-strip.kicad_pcb (KiCad board)
At the start: 2 copper layers, 202.4 x 15.4 mm, 36 parts

Commit message: Move LEDs to be properly on top of solenoids
Parts:
- moved R1 26.3 mm to (112.4, 130.8)
- moved R10 26.3 mm to (193.4, 130.8)
- moved R11 26.3 mm to (202.4, 130.8)
- moved R12 26.3 mm to (211.4, 130.8)
- moved R13 26.3 mm to (220.4, 130.8)
- moved R14 26.3 mm to (229.4, 130.8)
- moved R15 26.3 mm to (238.4, 130.8)
- moved R16 26.3 mm to (247.4, 130.8)
- moved R2 26.3 mm to (121.4, 130.8)
- moved R3 26.3 mm to (130.4, 130.8)
- moved R4 26.3 mm to (139.4, 130.8)
- moved R5 26.3 mm to (148.4, 130.8)
- moved R6 26.3 mm to (157.4, 130.8)
- moved R7 26.3 mm to (166.4, 130.8)
- moved R8 26.3 mm to (175.4, 130.8)
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Routing:
- net Net-(J3-Pin_5): track 168.8 -> 195.1 mm
- net Net-(J3-Pin_7): track 192.7 -> 219.0 mm
- net Net-(J3-Pin_6): track 180.9 -> 207.2 mm
- net Net-(J3-Pin_4): track 157.0 -> 183.3 mm
- net Net-(J3-Pin_2): track 133.2 -> 159.5 mm
- net Net-(J3-Pin_1): track 121.4 -> 147.7 mm
- net Net-(J1-Pin_9): track 95.2 -> 121.5 mm
- net Net-(J1-Pin_8): track 83.6 -> 109.9 mm
- net Net-(J1-Pin_6): track 61.0 -> 87.3 mm
- net Net-(J1-Pin_7): track 72.3 -> 98.6 mm
- net Net-(J1-Pin_5): track 49.7 -> 76.0 mm
- net Net-(J1-Pin_4): track 38.4 -> 64.7 mm
- net Net-(J1-Pin_3): track 27.1 -> 53.4 mm
- net Net-(J3-Pin_8): track 204.4 -> 230.7 mm
- net Net-(J3-Pin_3): track 145.2 -> 171.5 mm
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Other:
- board size 202.4 x 15.4 mm -> 226.2 x 15.4 mm
