File: ayab-shield/arduino_shield.kicad_pcb (KiCad board)
At the start: 2 copper layers, 73.1 x 53.3 mm, 35 parts, among them IC1 ULN2803A, IC2 ULN2803A, IC3 MCP2300X/P, IC4 MCP2300X/P, J1 Power, J2 Digital/PWM, J3 Analog, J4 Digital/PWM, X1 KLDX-0202-AC

Commit message: Move polarity symbol to ayab-library
Parts:
- G***: value LOGO -> Polarity_Center_Negative_2mm_SilkScreen; footprint LOGO -> ayab-library:Polarity_Center_Negative_2mm_SilkScreen
Changed lines of the file:
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@@
 		)
 	)
-	(footprint "LOGO"
+	(footprint "ayab-library:Polarity_Center_Negative_2mm_SilkScreen"
 		(layer "F.Cu")
 		(at 180.6 117.4 90)
@@
 			)
 		)
-		(property "Value" "LOGO"
+		(property "Value" "Polarity_Center_Negative_2mm_SilkScreen"
 			(at 0.75 0 90)
 			(layer "F.SilkS")
