File: ayab-sr-esp32/ayab-sr-esp32.kicad_pcb (KiCad board)
At the start: 2 copper layers, 64.5 x 83.1 mm, 64 parts, among them J1 USB_C_Receptacle_USB2.0_16P, J14 Conn_01x08, J2 USB_C_Receptacle_USB2.0_16P, J3 DIN-7, J4 Conn_01x02, Q1 BSS138, U1 CH224A, U10 AP2112K-3.3, U2 USBLC6-2SC6, U3 ESP32-S3-WROOM-1, U4 74AHCT1G125, U5 HS91L02W2C01, U6 TPS54202, U7 INA381A1, U8 74LVC125, U9 TPS54202

Commit message: AYAB-SR-ESP32: 5 V divider from JLCPCB basic parts
R13 (13.7k, C22793) was an extended part. The U9 feedback divider is now
R12/R13 = 75k/10k (C23242 and C25804, both basic):
- output: 0.596 V × (1 + 75/10) = 5.07 V (was 4.95 V)
- one fewer extended-part fee
- R13 shares the 10k reel already used by eight other resistors

No other extended part has a basic or preferred replacement with the same
footprint and rating.

Co-Authored-By: Claude Opus 5.5 <noreply@anthropic.com>
Claude-Session: https://claude.ai/code/session_013hjzppJpAsDjhGU3Z3soKr
Parts:
- R12: value 100k -> 75k
- R13: value 13.7k -> 10k
Changed lines of the file:
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@@
 			)
 		)
-		(property "Value" "13.7k"
+		(property "Value" "10k"
 			(at 0 1.43 90)
 			(layer "F.Fab")
@@
 			)
 		)
-		(property "LCSC" "C22793"
+		(property "LCSC" "C25804"
 			(at 0 0 90)
 			(unlocked yes)
@@
 			)
 		)
-		(property "Value" "100k"
+		(property "Value" "75k"
 			(at 0 1.43 90)
 			(layer "F.Fab")
@@
 			)
 		)
-		(property "LCSC" "C25803"
+		(property "LCSC" "C23242"
 			(at 0 0 90)
 			(unlocked yes)

Commit message: AYAB-SR-ESP32: fixed resistors instead of the RV1/RV2 trimmers
The two trimmers were JLCPCB extended parts ($3 each per order). Their
settings will be tuned on the silverreed shield; the starting values are
now fixed with basic 0603 resistors:
- RV1 -> R24 3.3k (C22978): U6 regulates at
  0.596 V x (100 + 3.3 + 4.7) / (3.3 + 4.7) = 8.05 V after an overcurrent.
  Reason: 0.9 A in a 7 ohm solenoid (cold) is 6.3 V, plus the carriage
  Darlington's VCE and the DIN cable.
- RV2 -> R25 10k (C25804) + R26 7.5k (C23234) between R9 82k and R23 27k:
  CMPREF = 3.3 V x 34.5 / 126.5 = 0.90 V, so the threshold is 0.90 A.

Board:
- R24 sits on RV1's pads.
- R25 and R26 sit in RV2's place.
- One GND stitching via was removed to make room.
- DRC still reports only the known U5 keep-out item.
- Net names follow the new parts: Net-(R24-Pad2), Net-(R25-Pad1).

Also: schematic notes, READMEs, fit check (no hand-made trimmer bodies),
production files, still renders.

Co-Authored-By: Claude Opus 5.5 <noreply@anthropic.com>
Claude-Session: https://claude.ai/code/session_013hjzppJpAsDjhGU3Z3soKr
Parts:
- removed RV1: 10k, Library:Potentiometer_Bourns_TC33X_Vertical
- removed RV2: 50k, Library:Potentiometer_Bourns_TC33X_Vertical
- added R24: 3.3k, Resistor_SMD:R_0603_1608Metric, F.Cu at (109.2, 81.9)
- added R25: 10k, Resistor_SMD:R_0603_1608Metric, F.Cu at (112.8, 78.0)
- added R26: 7.5k, Resistor_SMD:R_0603_1608Metric, F.Cu at (115.0, 79.7)
Routing:
- net /FB: track 48.0 -> 44.3 mm
- net Net-(R25-Pad1): track 28.2 -> 25.2 mm
- net GND: vias 275 -> 274
