File: ayab-sr-esp32/ayab-sr-esp32.kicad_sch (KiCad schematic)
At the start: 64 parts, among them J1 USB_C_Receptacle_USB2.0_16P, J14 Conn_01x08, J2 USB_C_Receptacle_USB2.0_16P, J3 DIN-7, J4 Conn_01x02, Q1 BSS138, U1 CH224A, U10 AP2112K-3.3, U2 USBLC6-2SC6, U3 ESP32-S3-WROOM-1, U4 74AHCT1G125, U5 HS91L02W2C01, U6 TPS54202, U7 INA381A1, U8 74LVC125, U9 TPS54202

Commit message: AYAB-SR-ESP32: mounting holes out of the JLCPCB BOM and placement files
H1-H3 are not placed parts: excluded from the BOM (schematic) and from the
BOM / position files (board), so JLCPCB no longer lists them as unmatched.
BOM, pick-and-place and JLCPCB CPL regenerated.

Co-Authored-By: Claude Opus 5.5 <noreply@anthropic.com>
Claude-Session: https://claude.ai/code/session_013hjzppJpAsDjhGU3Z3soKr
Parts:
- H1, H2, H3: now left out of the parts list
Changed lines of the file:
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@@
 		(body_style 1)
 		(exclude_from_sim no)
-		(in_bom yes)
+		(in_bom no)
 		(on_board yes)
 		(in_pos_files yes)
@@
 		(body_style 1)
 		(exclude_from_sim no)
-		(in_bom yes)
+		(in_bom no)
 		(on_board yes)
 		(in_pos_files yes)
@@
 		(body_style 1)
 		(exclude_from_sim no)
-		(in_bom yes)
+		(in_bom no)
 		(on_board yes)
 		(in_pos_files yes)

Commit message: AYAB-SR-ESP32: fix part rotations for JLCPCB assembly
JLCPCB's placement preview showed nine parts turned the wrong way. The
"FT Rotation Offset" field now corrects them in the CPL:
- U1, U2, U4, U7, U8: -90
- U6, U9: -90 (was +90, which put pin 1 on the opposite corner)
- U10 (AP2112K), Q1 (BSS138): 180

D1, D2, RV1, RV2, S1, J1 and J2 were already correct.

Co-Authored-By: Claude Opus 5.5 <noreply@anthropic.com>
Claude-Session: https://claude.ai/code/session_013hjzppJpAsDjhGU3Z3soKr
Parts:
- Q1, U10: FT Rotation Offset (none) -> 180
- U1, U2, U4, U7, U8: FT Rotation Offset (none) -> -90
- U6, U9: FT Rotation Offset 90 -> -90
Changed lines of the file:
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@@
 			)
 		)
+		(property "FT Rotation Offset" "180"
+			(at 326.39 74.93 0)
+			(hide yes)
+			(show_name no)
+			(do_not_autoplace no)
+			(effects
+				(font
+					(size 1.27 1.27)
+				)
+			)
+		)
 		(pin "2"
 		)
@@
 			)
 		)
-		(property "FT Rotation Offset" "90"
+		(property "FT Rotation Offset" "-90"
 			(at 57.15 142.24 0)
 			(hide yes)
@@
 			)
 		)
+		(property "FT Rotation Offset" "-90"
+			(at 228.6 149.86 0)
+			(hide yes)
+			(show_name no)
+			(do_not_autoplace no)
+			(effects
+				(font
+					(size 1.27 1.27)
+				)
+			)
+		)
 		(pin "1"
 		)
@@
 			)
 		)
+		(property "FT Rotation Offset" "-90"
+			(at 426.72 82.55 0)
+			(hide yes)
+			(show_name no)
+			(do_not_autoplace no)
+			(effects
+				(font
+					(size 1.27 1.27)
+				)
+			)
+		)
 		(pin "6"
 		)
@@
 			)
 		)
-		(property "FT Rotation Offset" "90"
+		(property "FT Rotation Offset" "-90"
 			(at 181.61 48.26 0)
 			(hide yes)
@@
 			)
 		)
+		(property "FT Rotation Offset" "-90"
+			(at 109.22 59.69 0)
+			(hide yes)
+			(show_name no)
+			(do_not_autoplace no)
+			(effects
+				(font
+					(size 1.27 1.27)
+				)
+			)
+		)
 		(pin "9"
 		)
@@
 			)
 		)
+		(property "FT Rotation Offset" "180"
+			(at 147.32 167.64 0)
+			(hide yes)
+			(show_name no)
+			(do_not_autoplace no)
+			(effects
+				(font
+					(size 1.27 1.27)
+				)
+			)
+		)
 		(pin "1"
 		)
@@
 			)
 		)
+		(property "FT Rotation Offset" "-90"
+			(at 265.43 269.24 0)
+			(hide yes)
+			(show_name no)
+			(do_not_autoplace no)
+			(effects
+				(font
+					(size 1.27 1.27)
+				)
+			)
+		)
 		(pin "5"
 		)
@@
 			(at 185.42 266.7 0)
 			(hide yes)
+			(show_name no)
+			(do_not_autoplace no)
+			(effects
+				(font
+					(size 1.27 1.27)
+				)
+			)
+		)
+		(property "FT Rotation Offset" "-90"
+			(at 185.42 266.7 0)
+			(hide yes)

Commit message: AYAB-SR-ESP32: R6 is a 50 mΩ part again in the BOM
R6, the INA381 current-sense shunt, is 50 mΩ in the schematic, but its
LCSC number C25334 is a 100 mΩ resistor (UNI-ROYAL 1206W4F100LT5E).
With that part, the over-current threshold would be halved.

Use C127691 instead: UNI-ROYAL 1206W3F500MT5E, 50 mΩ ±1%, 1/3 W, 1206.
It is an extended part at JLCPCB; no basic 50 mΩ part exists.

Co-Authored-By: Claude Opus 5.5 <noreply@anthropic.com>
Claude-Session: https://claude.ai/code/session_013hjzppJpAsDjhGU3Z3soKr
Parts:
- R6: LCSC C25334 -> C127691
Changed lines of the file:
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@@
 			)
 		)
-		(property "LCSC" "C25334"
+		(property "LCSC" "C127691"
 			(at 203.2 149.86 0)
 			(hide yes)

Commit message: AYAB-SR-ESP32: 5 V divider from JLCPCB basic parts
R13 (13.7k, C22793) was an extended part. The U9 feedback divider is now
R12/R13 = 75k/10k (C23242 and C25804, both basic):
- output: 0.596 V × (1 + 75/10) = 5.07 V (was 4.95 V)
- one fewer extended-part fee
- R13 shares the 10k reel already used by eight other resistors

No other extended part has a basic or preferred replacement with the same
footprint and rating.

Co-Authored-By: Claude Opus 5.5 <noreply@anthropic.com>
Claude-Session: https://claude.ai/code/session_013hjzppJpAsDjhGU3Z3soKr
Parts:
- R12: value 100k -> 75k; LCSC C25803 -> C23242
- R13: value 13.7k -> 10k; LCSC C22793 -> C25804
Changed lines of the file:
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@@
 			)
 		)
-		(property "Value" "13.7k"
+		(property "Value" "10k"
 			(at 229.87 86.36 0)
 			(show_name no)
@@
 			)
 		)
-		(property "LCSC" "C22793"
+		(property "LCSC" "C25804"
 			(at 224.79 85.09 0)
 			(hide yes)
@@
 			)
 		)
-		(property "Value" "100k"
+		(property "Value" "75k"
 			(at 229.87 60.96 0)
 			(show_name no)
@@
 			)
 		)
-		(property "LCSC" "C25803"
+		(property "LCSC" "C23242"
 			(at 224.79 59.69 0)
 			(hide yes)

Commit message: AYAB-SR-ESP32: fixed resistors instead of the RV1/RV2 trimmers
The two trimmers were JLCPCB extended parts ($3 each per order). Their
settings will be tuned on the silverreed shield; the starting values are
now fixed with basic 0603 resistors:
- RV1 -> R24 3.3k (C22978): U6 regulates at
  0.596 V x (100 + 3.3 + 4.7) / (3.3 + 4.7) = 8.05 V after an overcurrent.
  Reason: 0.9 A in a 7 ohm solenoid (cold) is 6.3 V, plus the carriage
  Darlington's VCE and the DIN cable.
- RV2 -> R25 10k (C25804) + R26 7.5k (C23234) between R9 82k and R23 27k:
  CMPREF = 3.3 V x 34.5 / 126.5 = 0.90 V, so the threshold is 0.90 A.

Board:
- R24 sits on RV1's pads.
- R25 and R26 sit in RV2's place.
- One GND stitching via was removed to make room.
- DRC still reports only the known U5 keep-out item.
- Net names follow the new parts: Net-(R24-Pad2), Net-(R25-Pad1).

Also: schematic notes, READMEs, fit check (no hand-made trimmer bodies),
production files, still renders.

Co-Authored-By: Claude Opus 5.5 <noreply@anthropic.com>
Claude-Session: https://claude.ai/code/session_013hjzppJpAsDjhGU3Z3soKr
Parts:
- removed RV1: 10k, Library:Potentiometer_Bourns_TC33X_Vertical, symbol Device:R_Potentiometer_Trim
- removed RV2: 50k, Library:Potentiometer_Bourns_TC33X_Vertical, symbol Device:R_Potentiometer_Trim
- added R24: 3.3k, Resistor_SMD:R_0603_1608Metric, symbol Device:R
- added R25: 10k, Resistor_SMD:R_0603_1608Metric, symbol Device:R
- added R26: 7.5k, Resistor_SMD:R_0603_1608Metric, symbol Device:R
Connections:
- net CMPREF: now also R25.2, R26.1
- net FB: now also R24.1
- net at R5.2: now also R24.2
- net at R9.2: now also R25.1
- net at R23.1: now also R26.2
Other:
- note added: "INA381A1 (amplifier + comparator): trips when I > V(CMPREF) / 1 V/A (20 V/V x 50 mOhm shunt) RESET to GND: transparent mode ALERT: open-drain, active low normal: high, Q1 on, U6 FB held low, Vout ~ VIN (~15 V) overcurrent: low, Q1 off, U6 regulates at 8 V V_HYS = 4 uA x (12.5k + R10) = 0.38 V, i.e. ~0.4 A (R10 82k) Threshold: R9 82k / R25 10k / R26 7.5k / R23 27k CMPREF = 3.3 * 34.5 / 126.5 = 0.9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"
- note added: "Vout = 0.596 * (R24+R5+R4) / (R24+R5) = 0.596 * (3.3+4.7+100) / (3.3+4.7) = 8.05V (0.9 A in a 7 ohm solenoid = 6.3 V, plus the carriage Darlington VCE and the DIN cable: ~8 V) Default: Q1 on holds FB low, Vout ~ VIN (~15 V bypass) Overcurrent: Q1 off, U6 regulates at 8 V"
- note removed: "INA381A1 (amplifier + comparator): trips when I > V(CMPREF) / 1 V/A (20 V/V x 50 mOhm shunt) RESET to GND: transparent mode ALERT: open-drain, active low normal: high, Q1 on, U6 FB held low, Vout ~ VIN (~15 V) overcurrent: low, Q1 off, U6 regulates at the RV1 setpoint V_HYS = 4 uA x (12.5k + R10) = 0.38 V, i.e. ~0.4 A (R10 82k) Threshold (RV2): R9 82k / RV2 50k / R23 27k CMPREF 0.56..1.60 V, i.e.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"
- note removed: "Vout = 0.596 * (RV1+R5+R4) / (RV1+R5) Vout_min = 0.596 * (10+4.7+100) / (10+4.7) = 4.65V Vout_max = 0.596 * (0+4.7+100) / (0+4.7) = 13.28V Default: Q1 on holds FB low, Vout ~ VIN (~15 V bypass) Overcurrent: Q1 off, U6 regulates at the RV1 setpoint"
- moved on the sheet: R23

Commit message: ayab-sr-esp32: OLED on a low-profile socket, enclosure post under its far end
- J15: 1x4 2.54 mm female socket, 5.0 mm high (HC-PM254-5.0H-1x4PZ-02A,
  LCSC C42163122), on U5's former pads. U5 keeps its symbol (BOM, LCSC
  C5248081) with a pad-less footprint (outline, courtyard, 3D model raised
  5 mm) and is left out of the placement file: it is plugged in by hand.
- New library footprints and a generated STEP model for the socket.
- 3.6 mm hole in the PCB under the OLED's far end (161.0, 32.3) for a
  post of the tray; one GND stitching via removed for edge clearance.
- Enclosure: updated for the 6 mm longer board (holes, USB-C), 3 mm post
  from the tray floor up to 0.1 mm under the module, lid ceiling raised
  by 5 mm (12.8 mm) to clear the OLED glass (11.74 mm). Fit check: no
  collision. Sections redone in the current board frame, plus one through
  the post.
- DRC 0, ERC 0, pad-net check OK; connectivity changes only by J15.
  Production files, renders and viewer regenerated.

Co-Authored-By: Claude Opus 5.5 <noreply@anthropic.com>
Claude-Session: https://claude.ai/code/session_013hjzppJpAsDjhGU3Z3soKr
Parts:
- added J15: HC-PM254-5.0H-1x4PZ-02A, Library:PinSocket_1x04_P2.54mm_Vertical_H5.0, symbol Connector:Conn_01x04_Socket
- U5: footprint Display:ER_OLEDM0.91_1x-I2C -> Library:OLED_0.91_128x32_I2C_Module_Socket_H5.0
Connections:
- net +3.3V: now also J15.2 (Pin_2)
- net GND: now also J15.1 (Pin_1)
- net SCL: now also J15.3 (Pin_3)
- net SDA: now also J15.4 (Pin_4)

Commit message: ayab-sr-esp32: CH224A off the I2C bus, PCB cut under the OLED end, rectangular support block
- U1 CFG2/CFG3 no longer on SCL/SDA (no-connect flags): single-resistor
  mode, R1 alone requests 15 V. The bus serves the OLED only, so the display
  works with only J2 plugged in (an unpowered CH224A would hold the bus at
  ~2 V). Old U1 SDA/SCL tracks removed. Sheet notes and README updated
  (pin map, firmware notes, J2-only operation and PD-adapter-in-J2 detection).
- PCB cut along the antenna cut-out line (x = 158.9) up to the top edge;
  the round post hole is gone. One off-board stitching via removed.
- Enclosure: the OLED's overhanging far end rests on a rectangular block of
  the tray (x 159.3-165.0, y 27.0-37.6, joined to the side wall, 0.1 mm
  under the module). Fit check: no collision. Renders and sections redone.
- DRC 0, ERC 0. Connectivity change: SCL/SDA lose U1.2/U1.3 only.

Co-Authored-By: Claude Opus 5.5 <noreply@anthropic.com>
Claude-Session: https://claude.ai/code/session_013hjzppJpAsDjhGU3Z3soKr
Connections:
- net SCL: no longer U1.2 (CFG2)
- net SDA: no longer U1.3 (CFG3)
- no-connect marks 27 -> 29
Other:
- note added: "CFG2/CFG3 not connected: single- resistor mode, I2C unused (the bus serves the OLED only). Unpowered (J2 only), the CH224A would pull the bus below VIH"
Changed lines of the file:
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@@
 			(justify left)
 		)
+	)	(text "CFG2/CFG3 not connected: single-\nresistor mode, I2C unused (the bus\nserves the OLED only). Unpowered\n(J2 only), the CH224A would pull\nthe bus below VIH"
+		(exclude_from_sim no)
+		(at 85.09 97.79 0)
+		(effects
+			(font
+				(size 1.27 1.27)
+			)
+			(justify left)
+		)
 	)
 	(text "Using the 3V3 rail as a voltage\nreference (assumed more\nprecise than the 5V rail)"
@@
 	(wire
 		(pts
-			(xy 119.38 64.77) (xy 125.73 64.77)
-		)
-		(stroke
-			(width 0)
-			(type default)
-		)
-	)
-	(wire
-		(pts
 			(xy 400.05 46.99) (xy 411.48 46.99)
 		)
@@
 	(wire
 		(pts
-			(xy 119.38 62.23) (xy 125.73 62.23)
-		)
-		(stroke
-			(width 0)
-			(type default)
-		)
-	)
-	(wire
-		(pts
 			(xy 312.42 48.26) (xy 312.42 72.39)
 		)
@@
 		)
 	)
-	(label "SDA"
-		(at 125.73 64.77 180)
-		(effects
-			(font
-				(size 1.27 1.27)
-			)
-			(justify right bottom)
-		)
-	)
 	(label "Vsol"
 		(at 213.36 170.18 180)
@@
 		)
 	)
-	(label "SCL"
-		(at 125.73 62.23 180)
-		(effects
-			(font
-				(size 1.27 1.27)
-			)
-			(justify right bottom)
-		)
-	)
 	(label "CCP_3V"
 		(at 44.45 288.29 0)
@@
 		)
 	)
+	(no_connect
+		(at 119.38 62.23)
+	)
+	(no_connect
+		(at 119.38 64.77)
+	)
 	(sheet_instances

Commit message: ayab-sr-esp32: OLED module U5 out of the JLCPCB BOM, assembly-time parts in the README
U5 stays on the board (outline, courtyard, 3D model on J15) but is excluded
from the BOM as well as the CPL: the module is bought separately and plugged
into J15 at assembly. README: assembly-time parts section (pin order, header,
pin trimming, support block). Connectivity identical; DRC/ERC 0. BOM, viewer
and enclosure outputs regenerated (fit check still covers U5: no collision).

Co-Authored-By: Claude Opus 5.5 <noreply@anthropic.com>
Claude-Session: https://claude.ai/code/session_013hjzppJpAsDjhGU3Z3soKr
Parts:
- U5: now left out of the parts list
Changed lines of the file:
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@@
 		(body_style 1)
 		(exclude_from_sim no)
-		(in_bom yes)
+		(in_bom no)
 		(on_board yes)
 		(in_pos_files no)
